Commit message: adding dimensions to tree structure

File: robot.urdf (robot description, URDF)
Before this commit: robot test_robot, 4 links, 3 joints
Joints:
- joint joint1: origin (none) -> xyz=5 3 0 rpy=0 0 0
- joint joint2: origin (none) -> xyz=-2 5 0 rpy=0 0 1.57
- joint joint3: origin (none) -> xyz=5 0 0 rpy=0 0 -1.57

Commit message: adding joint axes to finish the kinematic model. visualize the URDF using graphiz

File: robot.urdf (robot description, URDF)
Before this commit: robot test_robot, 4 links, 3 joints
Joints:
- joint joint1: axis (none) -> -0.9 0.15 0
- joint joint2: axis (none) -> -0.707 0.707 0
- joint joint3: axis (none) -> 0.707 -0.707 0
