Commit message: visual robot model

File: urdf/r2d2.urdf (robot description, URDF)
Before this commit: robot r2d2, 7 links, 6 joints
Links:
- removed link axis
- removed link box
- removed link leg1
- removed link leg2
- removed link rod
- added link eye; visual box size=.08 .08 .08
- added link eye_pole; visual cylinder length=0.3 radius=0.02
- added link left_foot; visual box size=.1 .4 .1
- added link left_front_wheel; visual cylinder length=.1 radius=.035
- added link left_leg; visual box size=.6 .2 .1
- added link left_rear_wheel; visual cylinder length=.1 radius=.035
- added link right_foot; visual box size=.1 .4 .1
- added link right_front_wheel; visual cylinder length=.1 radius=.035
- added link right_leg; visual box size=.6 .2 .1
- added link right_rear_wheel; visual cylinder length=.1 radius=.035
- link body: mass 1 -> None; geometry visual cylinder length=.6 radius=.2
- link head: mass 1 -> None; geometry visual sphere radius=.2
Joints:
- removed joint boxconnect
- removed joint leg1connect
- removed joint leg2connect
- removed joint periscope
- removed joint swivel
- removed joint tilt
- added joint body_to_left_leg: type fixed, parent body, child left_leg, origin xyz=-.22 0 .25
- added joint body_to_right_leg: type fixed, parent body, child right_leg, origin xyz=.22 0 .25
- added joint eye_extension: type fixed, parent head, child eye_pole, origin xyz=-.04 .1414 .1414 rpy=0 0 0
- added joint eye_pole_to_eye: type fixed, parent eye_pole, child eye
- added joint head_swivel: type fixed, parent body, child head, origin xyz=0 0 0.3
- added joint left_foot_to_front: type fixed, parent left_foot, child left_front_wheel, origin xyz=0 .13 -.05
- added joint left_foot_to_rear: type fixed, parent left_foot, child left_rear_wheel, origin xyz=0 -.13 -.05
- added joint left_leg_to_foot: type fixed, parent left_leg, child left_foot, origin xyz=0 0 -.6
- added joint right_foot_to_front: type fixed, parent right_foot, child right_front_wheel, origin xyz=0 .13 -.05
- added joint right_foot_to_rear: type fixed, parent right_foot, child right_rear_wheel, origin xyz=0 -.13 -.05
- added joint right_leg_to_foot: type fixed, parent right_leg, child right_foot, origin xyz=0 0 -.6

Commit message: trying to get joints to work...

File: urdf/r2d2.urdf (robot description, URDF)
Before this commit: robot r2d2, 12 links, 11 joints
Joints:
- joint head_swivel: origin xyz=0 0 0.3 -> xyz=0 0 .3

Commit message: Head swivel works

File: urdf/r2d2.urdf (robot description, URDF)
Before this commit: robot r2d2, 12 links, 11 joints
Joints:
- joint head_swivel: axis (none) -> 0 0 1; type fixed -> continuous

Commit message: periscope working

File: urdf/r2d2.urdf (robot description, URDF)
Before this commit: robot r2d2, 12 links, 11 joints
Joints:
- removed joint eye_extension
- added joint periscope: type prismatic, parent head, child eye_pole, origin xyz=-.04 .1414 .1414 rpy=0 0 0, axis 0 0 1, limit lower=0 upper=.29 effort=10 velocity=.5

Commit message: r2d2 walks

File: urdf/r2d2.urdf (robot description, URDF)
Before this commit: robot r2d2, 12 links, 11 joints
Joints:
- joint body_to_left_leg: limit (none) -> lower=-.2 upper=.2 effort=10 velocity=3.0; type fixed -> revolute
- joint body_to_right_leg: limit (none) -> lower=-.2 upper=.2 effort=10 velocity=3.0; type fixed -> revolute

Commit message: added collision and inertial properties to some body parts

File: urdf/r2d2.urdf (robot description, URDF)
Before this commit: robot r2d2, 12 links, 11 joints
Links:
- link body: mass None -> 10; geometry collision cylinder length=.6 radius=.2; visual cylinder length=.6 radius=.2
- link eye: mass None -> 0.2; geometry collision box size=.08 .08 .08; visual box size=.08 .08 .08
- link head: mass None -> 1; geometry collision sphere radius=.2; visual sphere radius=.2
- link left_leg: mass None -> 10; geometry collision box size=.6 .2 .1; visual box size=.6 .2 .1
- link right_leg: mass None -> 10; geometry collision box size=.6 .2 .1; visual box size=.6 .2 .1

Commit message: collision properties and made-up inertial values for all body parts

File: urdf/r2d2.urdf (robot description, URDF)
Before this commit: robot r2d2, 12 links, 11 joints
Links:
- link eye_pole: mass None -> 10
- link left_foot: mass None -> 10; geometry collision box size=.1 .4 .1; visual box size=.1 .4 .1
- link left_front_wheel: mass None -> 1; geometry collision cylinder length=.1 radius=.035; visual cylinder length=.1 radius=.035
- link left_rear_wheel: mass None -> 1; geometry collision cylinder length=.1 radius=.035; visual cylinder length=.1 radius=.035
- link right_foot: mass None -> 10; geometry collision box size=.1 .4 .1; visual box size=.1 .4 .1
- link right_front_wheel: mass None -> 1; geometry collision cylinder length=.1 radius=.035; visual cylinder length=.1 radius=.035
- link right_rear_wheel: mass None -> 1; geometry collision cylinder length=.1 radius=.035; visual cylinder length=.1 radius=.035

Commit message: computed inertia values for all body parts

File: urdf/r2d2.urdf (robot description, URDF)
Before this commit: robot r2d2, 12 links, 11 joints
Links:
- link body: mass 10 -> 203.5752
- link eye: mass 0.2 -> 1.3824
- link eye_pole: mass 10 -> 1.017876; geometry collision cylinder length=0.3 radius=0.02; visual cylinder length=0.3 radius=0.02
- link head: mass 1 -> 45.2389
- link left_foot: mass 10 -> 10.8
- link left_front_wheel: mass 1 -> 1.03908
- link left_leg: mass 10 -> 32.4
- link left_rear_wheel: mass 1 -> 1.03908
- link right_foot: mass 10 -> 10.8
- link right_front_wheel: mass 1 -> 1.03908
- link right_leg: mass 10 -> 32.4
- link right_rear_wheel: mass 1 -> 1.03908
